File: Hardware/Geiger_Counter.brd (EAGLE design)
At the start: 108 x 45.7 mm, 56 parts, among them Q1 MPSA42, Q2 MPSA18, Q3 MMBT4403, Q4 MPSA18, U10 FT232RL-BASICSSOP, U17 AVR_SPI_PRG_6PTH, U7 TRANSFORMERAUDIO, U8 ATMEGA168, X1 USBSMD

Commit message: Schematic Cleanup / Trace redo
Parts:
- FRAME1: value FRAME-LETTER -> FRAME-LEDGER
Routing:
- net RST: track 108.2 -> 106.8 mm
- net HV: track 49.2 -> 50.3 mm
Changed lines of the file:
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@@
 <setting verticaltext="up"/>
 </settings>
-<grid distance="0.05" unitdist="inch" unit="inch" style="lines" multiple="1" display="yes" altdistance="0.001" altunitdist="inch" altunit="inch"/>
+<grid distance="0.05" unitdist="inch" unit="inch" style="lines" multiple="1" display="yes" altdistance="0.005" altunitdist="inch" altunit="inch"/>
 <layers>
 <layer number="1" name="Top" color="4" fill="1" visible="yes" active="yes"/>
@@
 <layer number="47" name="Measures" color="7" fill="1" visible="no" active="yes"/>
 <layer number="48" name="Document" color="7" fill="1" visible="no" active="yes"/>
-<layer number="49" name="Reference" color="7" fill="1" visible="yes" active="yes"/>
+<layer number="49" name="Reference" color="7" fill="1" visible="no" active="yes"/>
 <layer number="50" name="dxf" color="7" fill="1" visible="no" active="yes"/>
 <layer number="51" name="tDocu" color="6" fill="1" visible="yes" active="yes"/>
@@
 <element name="JP1" library="SparkFun" package="MICRO-FIDUCIAL" value="FIDUCIALUFIDUCIAL" x="6.35" y="2.54"/>
 <element name="JP3" library="SparkFun" package="MICRO-FIDUCIAL" value="FIDUCIALUFIDUCIAL" x="102.87" y="44.45"/>
-<element name="FRAME1" library="SparkFun-Aesthetics" package="CREATIVE_COMMONS" value="FRAME-LETTER" x="21.78894375" y="-19.05"/>
+<element name="FRAME1" library="SparkFun-Aesthetics" package="CREATIVE_COMMONS" value="FRAME-LEDGER" x="21.78894375" y="-19.05"/>
 </elements>
 <signals>
@@
 <contactref element="C6" pad="1"/>
 <contactref element="S1" pad="C@2"/>
-<wire x1="39.37" y1="34.29" x2="45.72" y2="27.94" width="0.6096" layer="16"/>
-<wire x1="39.37" y1="34.518" x2="39.37" y2="34.29" width="0.6096" layer="16"/>
 <contactref element="R8" pad="P$1"/>
 <wire x1="76.454" y1="25.4" x2="76.454" y2="30.226" width="0.6096" layer="16"/>
 <wire x1="76.454" y1="30.226" x2="76.2" y2="30.48" width="0.6096" layer="16"/>
-<wire x1="57.15" y1="25.4" x2="57.15" y2="27.94" width="0.6096" layer="16"/>
-<wire x1="57.15" y1="27.94" x2="57.15" y2="29.21" width="0.6096" layer="16"/>
+<wire x1="57.15" y1="25.4" x2="57.15" y2="29.21" width="0.6096" layer="16"/>
 <wire x1="57.15" y1="29.21" x2="58.42" y2="30.48" width="0.6096" layer="16"/>
 <wire x1="58.42" y1="30.48" x2="76.2" y2="30.48" width="0.6096" layer="16"/>
-<wire x1="45.72" y1="27.94" x2="57.15" y2="27.94" width="0.6096" layer="16"/>
+<wire x1="39.37" y1="34.29" x2="46.863" y2="26.797" width="0.6096" layer="16"/>
+<wire x1="46.863" y1="26.797" x2="54.102" y2="26.797" width="0.6096" layer="16"/>
+<wire x1="54.102" y1="26.797" x2="55.499" y2="25.4" width="0.6096" layer="16"/>
+<wire x1="55.499" y1="25.4" x2="57.15" y2="25.4" width="0.6096" layer="16"/>
+<wire x1="39.37" y1="34.29" x2="39.37" y2="34.518" width="0.6096" layer="16"/>
 </signal>
 <signal name="N$14">
@@
 <wire x1="13.57" y1="14.116" x2="13.57" y2="16.4846" width="0.254" layer="1"/>
 <wire x1="13.589" y1="14.097" x2="13.57" y2="14.116" width="0.254" layer="1"/>
-<wire x1="6.858" y1="3.81" x2="15.24" y2="3.81" width="0.254" layer="16"/>
+<wire x1="6.858" y1="3.81" x2="12.7" y2="3.81" width="0.254" layer="16"/>
+<wire x1="12.7" y1="3.81" x2="15.24" y2="3.81" width="0.254" layer="16"/>
 <wire x1="5.715" y1="4.953" x2="6.858" y2="3.81" width="0.254" layer="16"/>
 <wire x1="16.51" y1="2.54" x2="19.05" y2="2.54" width="0.3556" layer="1"/>
@@
 <wire x1="20.828" y1="23.026" x2="20.74" y2="23.114" width="0.254" layer="1"/>
 <wire x1="13.589" y1="14.097" x2="13.589" y2="12.7" width="0.254" layer="16"/>
-<wire x1="13.589" y1="12.7" x2="13.589" y2="12.319" width="0.254" layer="16"/>
-<wire x1="13.589" y1="12.319" x2="6.35" y2="5.08" width="0.254" layer="16"/>
 <wire x1="6.35" y1="5.08" x2="5.842" y2="5.08" width="0.254" layer="16"/>
 <wire x1="5.842" y1="5.08" x2="5.715" y2="4.953" width="0.254" layer="16"/>
 <wire x1="20.701" y1="12.827" x2="13.716" y2="12.827" width="0.254" layer="16"/>
 <wire x1="13.716" y1="12.827" x2="13.589" y2="12.7" width="0.254" layer="16"/>
+<wire x1="13.589" y1="12.7" x2="13.589" y2="7.239" width="0.254" layer="16"/>
+<wire x1="13.589" y1="7.239" x2="12.7" y2="6.35" width="0.254" layer="16"/>
+<wire x1="12.7" y1="6.35" x2="12.7" y2="3.81" width="0.254" layer="16"/>
 </signal>
 <signal name="MOSI">
